Commit message: Fix: Gazebo working with NVIDIA GPU, green lane, colored obstacles, sensors

File: src/adas_robot_description/urdf/urdf_latest.urdf (robot description, URDF)
Before this commit: robot urdf_latest, 11 links, 10 joints
Joints:
- joint leftfront: axis 0 0 -1 -> (none); limit effort=10 velocity=10 -> (none); type continuous -> fixed
- joint leftfrontknuckle: axis 0 0 1 -> (none); limit effort=10 velocity=10 -> (none); type continuous -> fixed
- joint rightfront: axis 0 0 1 -> (none); limit effort=10 velocity=10 -> (none); type continuous -> fixed
- joint rightfrontknuckle: axis 0 0 1 -> (none); limit effort=10 velocity=10 -> (none); type continuous -> fixed

Commit message: Fix: Both rear wheel axes aligned, robot moves straight

File: src/adas_robot_description/urdf/urdf_latest.urdf (robot description, URDF)
Before this commit: robot urdf_latest, 11 links, 10 joints
Joints:
- joint leftrear: axis 0 0 -1 -> 0 0 1
